Commit message: fix lenght values

File: src/three_finger_hand/urdf/finger.xacro (robot description, xacro)
@@ -32,5 +32,5 @@
       <parent link="${prefix}_knuckle"/>
       <child link="${prefix}_proximal"/>
-      <origin xyz="0 0 0.07" rpy="0 0 1.57"/>
+      <origin xyz="0 0 0.01025" rpy="0 0 1.57"/>
       <axis xyz="1 0 0"/> <limit lower="-1.57" upper="1.57" effort="10" velocity="1.0"/>
     </joint>
@@ -57,5 +57,5 @@
       <parent link="${prefix}_proximal"/>
       <child link="${prefix}_middle"/>
-      <origin xyz="0 0 0.01025" rpy="0 0 -1.57"/>
+      <origin xyz="0 0 0.07" rpy="0 0 -1.57"/>
       <axis xyz="0 1 0"/>
       <limit lower="-1.57" upper="1.57" effort="10" velocity="1.0"/>

Commit message: add gui controller file, edit joint limits to solve mechanical problems

File: src/three_finger_hand/urdf/finger.xacro (robot description, xacro)
@@ -6,5 +6,7 @@
       <child link="${prefix}_knuckle"/>
       <xacro:insert_block name="origin"/>
-      <axis xyz="1 0 0"/> <limit lower="-1.57" upper="1.57" effort="10" velocity="1.0"/>
+      <axis xyz="1 0 0"/> <limit lower="-1.256" upper="1.256" effort="10" velocity="1.0"/>
+      <damping value="0.5"/>
+      <dynamics friction="0.5"/>
     </joint>
     <link name="${prefix}_knuckle">
@@ -25,6 +27,6 @@
       </collision>
       <inertial>
-        <mass value="0.05"/>
-        <inertia ixx="0.0001" ixy="0" ixz="0" iyy="0.0001" iyz="0" izz="0.0001"/>
+        <mass value="0.03"/>
+        <inertia ixx="0.005" ixy="0" ixz="0" iyy="0.005" iyz="0" izz="0.005"/>
       </inertial>
     </link>
@@ -33,5 +35,7 @@
       <child link="${prefix}_proximal"/>
       <origin xyz="0 0 0.01025" rpy="0 0 1.57"/>
-      <axis xyz="1 0 0"/> <limit lower="-1.57" upper="1.57" effort="10" velocity="1.0"/>
+      <axis xyz="1 0 0"/> <limit lower="-0.628" upper="1.256" effort="10" velocity="1.0"/>
+      <damping value="0.5"/>
+      <dynamics friction="0.5"/>
     </joint>
     <link name="${prefix}_proximal">
@@ -51,5 +55,5 @@
       <inertial>
         <mass value="0.05"/>
-        <inertia ixx="0.0001" ixy="0" ixz="0" iyy="0.0001" iyz="0" izz="0.0001"/>
+        <inertia ixx="0.005" ixy="0" ixz="0" iyy="0.005" iyz="0" izz="0.005"/>
       </inertial>
     </link>
@@ -59,5 +63,7 @@
       <origin xyz="0 0 0.07" rpy="0 0 -1.57"/>
       <axis xyz="0 1 0"/>
-      <limit lower="-1.57" upper="1.57" effort="10" velocity="1.0"/>
+      <limit lower="-1.256" upper="1.256" effort="10" velocity="1.0"/>
+      <damping value="0.5"/>
+      <dynamics friction="0.5"/>
     </joint>
     <link name="${prefix}_middle">
@@ -77,5 +83,5 @@
       <inertial>
         <mass value="0.04"/>
-        <inertia ixx="0.0001" ixy="0" ixz="0" iyy="0.0001" iyz="0" izz="0.0001"/>
+        <inertia ixx="0.005" ixy="0" ixz="0" iyy="0.005" iyz="0" izz="0.005"/>
       </inertial>
     </link>
@@ -86,4 +92,6 @@
       <axis xyz="0 1 0"/>
       <limit lower="-1.57" upper="1.57" effort="10" velocity="1.0"/>
+      <damping value="0.5"/>
+      <dynamics friction="0.5"/>
     </joint>
     <link name="${prefix}_distal">
@@ -102,6 +110,6 @@
       </collision>
       <inertial>
-        <mass value="0.03"/>
-        <inertia ixx="0.0001" ixy="0" ixz="0" iyy="0.0001" iyz="0" izz="0.0001"/>
+        <mass value="0.02"/>
+        <inertia ixx="0.005" ixy="0" ixz="0" iyy="0.005" iyz="0" izz="0.005"/>
       </inertial>
     </link>

File: src/three_finger_hand/urdf/three_finger_hand.urdf.xacro (robot description, xacro)
@@ -25,5 +25,5 @@
     </collision>
     <inertial>
-      <mass value="0.5"/>
+      <mass value="0.7"/>
       <inertia ixx="0.001" ixy="0" ixz="0" iyy="0.001" iyz="0" izz="0.001"/>
     </inertial>
@@ -49,60 +49,96 @@
     </hardware>
     <joint name="finger_1_joint_1">
-      <command_interface name="position"><param name="min">-1.57</param><param name="max">1.57</param></command_interface>
+      <command_interface name="position">
+        <param name="min">-1.256</param>
+        <param name="max">1.256</param>
+      </command_interface>
       <state_interface name="position"/>
       <state_interface name="velocity"/>
     </joint>
     <joint name="finger_1_joint_2">
-      <command_interface name="position"><param name="min">0.0</param><param name="max">1.57</param></command_interface>
+      <command_interface name="position">
+        <param name="min">-0.628</param>
+        <param name="max">1.256</param>
+      </command_interface>
       <state_interface name="position"/>
       <state_interface name="velocity"/>
     </joint>
     <joint name="finger_1_joint_3">
-      <command_interface name="position"><param name="min">0.0</param><param name="max">1.57</param></command_interface>
+      <command_interface name="position">
+        <param name="min">-1.256</param>
+        <param name="max">1.256</param>
+      </command_interface>
       <state_interface name="position"/>
       <state_interface name="velocity"/>
     </joint>
     <joint name="finger_1_joint_4">
-      <command_interface name="position"><param name="min">0.0</param><param name="max">1.57</param></command_interface>
+      <command_interface name="position">
+        <param name="min">-1.57</param>
+        <param name="max">1.57</param>
+      </command_interface>
       <state_interface name="position"/>
       <state_interface name="velocity"/>
     </joint>
     <joint name="finger_2_joint_1">
-      <command_interface name="position"><param name="min">-1.57</param><param name="max">1.57</param></command_interface>
+      <command_interface name="position">
+        <param name="min">-1.256</param>
+        <param name="max">1.256</param>
+      </command_interface>
       <state_interface name="position"/>
       <state_interface name="velocity"/>
     </joint>
     <joint name="finger_2_joint_2">
-      <command_interface name="position"><param name="min">0.0</param><param name="max">1.57</param></command_interface>
+      <command_interface name="position">
+        <param name="min">-0.628</param>
+        <param name="max">1.256</param>
+      </command_interface>
       <state_interface name="position"/>
       <state_interface name="velocity"/>
     </joint>
     <joint name="finger_2_joint_3">
-      <command_interface name="position"><param name="min">0.0</param><param name="max">1.57</param></command_interface>
+      <command_interface name="position">
+        <param name="min">-1.256</param>
+        <param name="max">1.256</param>
+      </command_interface>
       <state_interface name="position"/>
       <state_interface name="velocity"/>
     </joint>
     <joint name="finger_2_joint_4">
-      <command_interface name="position"><param name="min">0.0</param><param name="max">1.57</param></command_interface>
+      <command_interface name="position">
+        <param name="min">-1.57</param>
+        <param name="max">1.57</param>
+      </command_interface>
       <state_interface name="position"/>
       <state_interface name="velocity"/>
     </joint>
     <joint name="finger_3_joint_1">
-      <command_interface name="position"><param name="min">-1.57</param><param name="max">1.57</param></command_interface>
+      <command_interface name="position">
+        <param name="min">-1.256</param>
+        <param name="max">1.256</param>
+      </command_interface>
       <state_interface name="position"/>
       <state_interface name="velocity"/>
     </joint>
     <joint name="finger_3_joint_2">
-      <command_interface name="position"><param name="min">0.0</param><param name="max">1.57</param></command_interface>
+      <command_interface name="position">
+        <param name="min">-0.628</param>
+        <param name="max">1.256</param>
+      </command_interface>
       <state_interface name="position"/>
       <state_interface name="velocity"/>
     </joint>
     <joint name="finger_3_joint_3">
-      <command_interface name="position"><param name="min">0.0</param><param name="max">1.57</param></command_interface>
+      <command_interface name="position">
+        <param name="min">-1.256</param>
+        <param name="max">1.256</param>
+      </command_interface>
       <state_interface name="position"/>
       <state_interface name="velocity"/>
     </joint>
     <joint name="finger_3_joint_4">
-      <command_interface name="position"><param name="min">0.0</param><param name="max">1.57</param></command_interface>
+      <command_interface name="position">
+        <param name="min">-1.57</param>
+        <param name="max">1.57</param>
+      </command_interface>
       <state_interface name="position"/>
       <state_interface name="velocity"/>
